Commit message: 雷达盲区实测与配套工具 (VLP-16)
- scripts/lidar_blind_zone.py: 抓一帧点云按 地面/本体/环境/无回波 分类, 输出逐扫描线统计、
  盲区锥面公式与逐高度可见性表
- scripts/lidar_target_check.py: 近场靶标校验, 自动判定 0.5 m 最小量程边界
- scripts/lidar_capture_png.py: 点云出图(俯视+3D 双面板), 需 matplotlib
- worlds/lidar_blindzone_targets.sdf: 0.40/0.48/0.52/0.68 m 四块靶板
- README 七.7: 三种姿态实测结论 —— 本体自遮挡 0 条射线; 近场地面盲环半径 3.39 m;
  靶标校验 4/4 通过(0.527 / 0.684 m 与几何值吻合)
- .gitignore: 忽略出图默认输出 vlp16_scan.png

File: urdf/AG_robot.urdf.xacro (robot description, xacro)
@@ -20,5 +20,7 @@
           │     ├─ arm1_*          松灵 PiPER
           │     └─ arm2_*          松灵 PiPER
-     激光雷达与相机: 位置未定, 本次没有加 (urdf/sensors_disabled.xacro 里留了完整定义)。
+     传感器:
+       Velodyne VLP-16 3D 激光雷达暂用圆柱体代替正式网格，固定在立柱顶部正中心。
+       相机位置仍未确定，旧定义保留在 urdf/sensors_disabled.xacro 中但不启用。
      ===================================================================== -->
 <robot name="AG_robot" xmlns:xacro="http://www.ros.org/wiki/xacro">
@@ -52,4 +54,5 @@
   <material name="alu"><color rgba="0.78 0.79 0.81 1.0"/></material>
   <material name="dark"><color rgba="0.22 0.22 0.24 1.0"/></material>
+  <material name="velodyne_blue"><color rgba="0.05 0.22 0.42 1.0"/></material>
   <!-- piper_arm.xacro 的 link2/link5 引用 accent, 本包必须自己定义一份,
        否则 urdf 解析会报 "material 'accent' undefined" 并退回 RViz 默认色。
@@ -276,4 +279,31 @@
     </inertial>
   </link>
+  <!-- ═════════ Velodyne VLP-16 3D 激光雷达（临时几何）═════════
+       2026-09-25 实测 base_frame.stl 包围盒：
+         X = [-0.250, 0.250] m，Y = [-0.174797, -0.055] m，Z 顶面 = 0.911 m。
+       因此安装中心暂定为 (0, -0.114898, 0.947)：圆柱高 72 mm，底面正好落在立柱顶面。
+       直径 89 mm、高 72 mm、质量 0.59 kg 取自当前 VLP-16 官方规格页。
+       正式 CAD / mesh 完成后，只需替换本 link 的 visual/collision 并修正 joint origin。
+       Gazebo 的 16 线扫描器定义在 urdf/gazebo.xacro。 -->
+  <link name="velodyne_link">
+    <visual>
+      <geometry><cylinder radius="0.0445" length="0.072"/></geometry>
+      <material name="velodyne_blue"/>
+    </visual>
+    <collision>
+      <geometry><cylinder radius="0.0445" length="0.072"/></geometry>
+    </collision>
+    <inertial>
+      <origin xyz="0 0 0" rpy="0 0 0"/>
+      <mass value="0.59"/>
+      <inertia ixx="0.000547" ixy="0" ixz="0"
+               iyy="0.000547" iyz="0" izz="0.000584"/>
+    </inertial>
+  </link>
+  <joint name="velodyne_joint" type="fixed">
+    <parent link="base_frame_link"/>
+    <child link="velodyne_link"/>
+    <origin xyz="0 -0.114898 0.947" rpy="0 0 0"/>
+  </joint>
   <!-- ═════════ 两条松灵 PiPER 六轴臂 ═════════
        臂本体参数取自官方 agx_arm_urdf/piper (见 urdf/piper_arm.xacro), 网格是米制不用 scale。
@@ -305,8 +335,5 @@
     <origin xyz="-0.190000 -0.247667 0.032000" rpy="0 0 -1.5707963"/>
   </xacro:piper_arm>
-  <!-- ═════════ 激光雷达 / 相机: 位置未定, 本次不加 ═════════
-       完整定义在 urdf/sensors_disabled.xacro, 网格 car_laser.stl / car_camera_link.stl 也在 meshes/ 下。
-       解开下面这行 include 即可接回来:
-       <xacro:include filename="$(find ag_robot_description)/urdf/sensors_disabled.xacro"/> -->
+  <!-- 旧版 2D 雷达 / 相机定义保留在 urdf/sensors_disabled.xacro，本模型不启用。 -->
   <!-- <gazebo reference="base_link"><material>Gazebo/Grey</material></gazebo>   (已由 .obj 自带颜色取代; 若 Gazebo 不认 .obj 材质, 把这几行解开即可) -->
   <xacro:macro name="wheel_gz" params="i">

File: urdf/gazebo.xacro (robot description, xacro)
@@ -70,3 +70,44 @@
   <xacro:wheel_gz i="1"/><xacro:wheel_gz i="2"/>
   <xacro:wheel_gz i="3"/><xacro:wheel_gz i="4"/>
+  <!-- Velodyne VLP-16 临时仿真参数（当前官方 VLP-16 规格）：
+       16 线，水平 360°，垂直 40°，最大量程 200 m，精度 ±3 cm，最高 20 Hz。
+       本仿真采用 10 Hz × 1800 水平采样 × 16 线 = 288000 点/秒；
+       需要模拟最大帧率时可把 update_rate 改为 20（约 576000 点/秒）。 -->
+  <gazebo reference="velodyne_link">
+    <sensor name="velodyne_vlp16" type="gpu_lidar">
+      <pose>0 0 0.010 0 0 0</pose>
+      <topic>velodyne/scan</topic>
+      <gz_frame_id>velodyne_link</gz_frame_id>
+      <update_rate>10</update_rate>
+      <always_on>true</always_on>
+      <visualize>true</visualize>
+      <lidar>
+        <scan>
+          <horizontal>
+            <samples>1800</samples>
+            <resolution>1</resolution>
+            <min_angle>-${pi}</min_angle>
+            <max_angle>${pi}</max_angle>
+          </horizontal>
+          <vertical>
+            <samples>16</samples>
+            <resolution>1</resolution>
+            <min_angle>-0.34906585</min_angle>
+            <max_angle>0.34906585</max_angle>
+          </vertical>
+        </scan>
+        <range>
+          <min>0.5</min>
+          <max>200.0</max>
+          <resolution>0.01</resolution>
+        </range>
+        <noise>
+          <type>gaussian</type>
+          <mean>0.0</mean>
+          <!-- 官方 ±3 cm 精度近似为高斯噪声的 ±3σ，因此 σ 取 1 cm。 -->
+          <stddev>0.01</stddev>
+        </noise>
+      </lidar>
+    </sensor>
+  </gazebo>
 </robot>

Commit message: 雷达姿态参数化: 一个 lidar_pitch 参数切换四种安装倾角 (0/15/25/35)
原来四种姿态是三个写死倾角的提交 + 手工改靶板 SDF 的 pose, 下游要逐个 checkout 重编。
现在:
- urdf/AG_robot.urdf.xacro: 新增 xacro 参数 lidar_pitch (度, 正值=朝车头 base_frame_link -Y
  下倾), 驱动 velodyne_joint 的 roll 与安装高度 z = 0.911 + 0.036cos + 0.0445sin (倾斜圆柱最低
  外缘必须仍落在立柱顶面, 否则穿模); 0/15/25/35 四档数值与历史标签 vlp16-level-0deg /
  vlp16-tilt15 / vlp16-tilt25 / vlp16-tilt35 逐值一致
- launch: gazebo.launch.py 与 display.launch.py 透传 lidar_pitch 并打印当前姿态
- scripts/lidar_blind_zone.py: 倾角与安装高度改为从 TF 读 (支持任意姿态), 保留解析地面平面
  判定与逐方向下视角/车尾扇区输出
- scripts/spawn_lidar_targets.py: 按 TF 自动算靶板位姿, 任意倾角都与雷达光心对齐
- scripts/lidar_pose_sweep.sh: 四姿态依次起仿真测盲区并输出对比表 (自动撤演示障碍物 + 污染自查)
- docs/lidar_poses/: 四姿态点云俯视图
- README 七.8: 四姿态实测对比表、选型建议、SLAM 侧接法与前置条件 (IMU 传感器 / /imu/data
  桥接 / robot_localization EKF + enable_odom_tf 改 false)

实测 (与历史记录交叉验证一致): 0° 车头 3.22 m 全向对称; 15° 车头 1.69 / 左右 3.37 / 车尾 13.40;
25° 车头 1.19、车尾无地面扇区 77.38°; 35° 车头 0.83 / 左右 4.08、车尾扇区 117.36°
(与历史记录 0.830-0.831 / 4.083-4.104 / 117.36° 一致); 四种姿态本体自遮挡均为 0 条射线

File: urdf/AG_robot.urdf.xacro (robot description, xacro)
@@ -42,4 +42,18 @@
   <xacro:arg name="arm1_prefix" default="arm1_"/>
   <xacro:arg name="arm2_prefix" default="arm2_"/>
+  <!-- ═════════ 雷达安装倾角（参数化, 供 SLAM 对比四种姿态）═════════
+       lidar_pitch 单位: 度; 正值 = 朝车头方向(base_frame_link 的 -Y)下倾。
+       已验证 0(水平) / 15 / 25 / 35, 实际填任意角度都行。
+       切换方式: ros2 launch ag_robot_description gazebo.launch.py lidar_pitch:=25
+       —— xacro 在 launch 时才展开, 所以换角度不需要重新 colcon build。
+       joint 的 z 必须随倾角抬高, 否则倾斜圆柱的最低外缘会插进立柱顶面(z=0.911 m):
+           z(pitch) = 0.911 + (h/2)·cos(pitch) + r·sin(pitch),  h=0.072, r=0.0445
+       取值: 0°→0.947(水平版原值)  15°→0.9573  25°→0.9624  35°→0.9660
+             (35° 与历史提交 vlp16-tilt35 的 0.966013 一致) -->
+  <xacro:arg name="lidar_pitch" default="0"/>
+  <xacro:property name="lidar_pitch_deg" value="$(arg lidar_pitch)"/>
+  <xacro:property name="lidar_pitch_rad" value="${radians(float(lidar_pitch_deg))}"/>
+  <xacro:property name="velodyne_z"
+                  value="${0.911 + 0.036*cos(lidar_pitch_rad) + 0.0445*sin(lidar_pitch_rad)}"/>
   <xacro:property name="arm1_prefix" value="$(arg arm1_prefix)"/>
   <xacro:property name="arm2_prefix" value="$(arg arm2_prefix)"/>
@@ -304,5 +318,6 @@
     <parent link="base_frame_link"/>
     <child link="velodyne_link"/>
-    <origin xyz="0 -0.114898 0.947" rpy="0 0 0"/>
+    <!-- 位姿由 lidar_pitch 参数驱动, 见文件开头那段注释 -->
+    <origin xyz="0 -0.114898 ${velodyne_z}" rpy="${lidar_pitch_rad} 0 0"/>
   </joint>
   <!-- ═════════ 两条松灵 PiPER 六轴臂 ═════════

Commit message: urdf: 双臂加装 PiPER 官方平行夹爪 (mimic 联动, 控制器 5 -> 7)
两条 PiPER 六轴臂末端按官方定义挂上平行夹爪。几何、惯性、安装位姿与限位取自
agx_arm_urdf/piper/urdf/piper_with_gripper_description.xacro。

模型: 28 link / 27 关节 -> 36 link / 35 关节 (12 固定 + 4 连续 + 12 旋转 + 7 平移)
- 每臂新增 4 个 link: gripper_base / gripper_link / gripper_link1 / gripper_link2
- arm{1,2}_gripper 是唯一主动关节 (prismatic, 0..0.10 m), 位置值表示两指总开口宽度:
  0 = 完全闭合, 0.10 m = 完全打开
- 两根指爪 gripper_joint1/2 由 <mimic> 分别以 +0.5 / -0.5 倍联动
- 保留 arm{1,2}_tool0 法兰外端面 frame 名, 现有规划与 TF 用户不受影响

两处踩过的坑, 都写进注释了:
- link gripper_link 补 0.001 kg 虚拟惯量: 官方显示模型把该 link 定义成空 link, 而
  sdformat 会删除"没有 inertial 的可动 link", 连带删掉 gripper 主关节, 后面两个 mimic
  关节就找不到驱动源。实体夹爪质量仍是 0.45 + 0.025 + 0.025 = 0.50 kg。
- gazebo.launch.py 显式指定 --physics-engine gz-physics-bullet-featherstone-plugin:
  Harmonic 默认的 DART 不支持 SDF mimic constraint, 夹爪两指联动会失效。

控制器: 5 -> 7 个。新增 arm1_gripper_controller / arm2_gripper_controller, 都是
JointTrajectoryController (position 命令 + position/velocity 状态, 容差 trajectory 0.01 /
goal 0.002)。gazebo.xacro 只给 gripper 主关节开命令接口, 两根指爪只暴露状态接口; 不走
gz_ros2_control 的 mimic 参数, 否则当前 Humble 插件会把 /joint_states 里的关节名改成
*_mimic, robot_state_publisher 就更新不了指爪 TF。

网格: 新增 6 个 (夹爪 visual .dae / collision .stl 各 3 个, 共约 4.5 MB), meshes/ 从
26 个增至 32 个; NOTICE 补上这三组网格的署名 (同样来自 AgileX agx_arm_urdf, MIT)。

验证:
- xacro 展开 + check_urdf: Successfully Parsed XML, base_footprint 单一根节点
- link/joint 计数与 README 声称一致 (36 / 35, 类型分布 12+4+12+7)
- 模型引用的 30 个网格逐个核对, 0 缺失; 未被引用的仍只有 car_camera_link / car_laser
- 新 .dae 为合法 XML; 新 .stl 头部三角面数与文件尺寸自洽 (36756 / 2086 / 2086)

README 同步更新: 模型结构树、能力表、目录结构、控制器数量、网格计数。

File: urdf/AG_robot.urdf.xacro (robot description, xacro)
@@ -18,6 +18,6 @@
           ├─ base_frame_link       立柱+导轨+推杆 (固定)
           │  └─ lift_platform_link 升降台, 沿立柱 Z 向滑动
-          │     ├─ arm1_*          松灵 PiPER
-          │     └─ arm2_*          松灵 PiPER
+          │     ├─ arm1_*          松灵 PiPER + 平行夹爪
+          │     └─ arm2_*          松灵 PiPER + 平行夹爪
      传感器:
        Velodyne VLP-16 3D 激光雷达暂用圆柱体代替正式网格，固定在立柱顶部正中心。

File: urdf/gazebo.xacro (robot description, xacro)
@@ -32,4 +32,30 @@
     <xacro:iface_pos name="${prefix}joint6"/>
   </xacro:macro>
+  <!-- PiPER 夹爪的主关节表示两指总开口宽度（0..0.10 m）。
+       两个指爪关节是 mimic 从关节，仅暴露原名状态接口，不单独接受命令。
+       联动由 URDF <mimic> 转换出的 SDF mimic constraint 完成，所以这里不再写
+       gz_ros2_control 的 mimic 参数。否则当前 Humble 插件会把 /joint_states 中的
+       关节改名为 *_mimic，导致 robot_state_publisher 无法更新指爪 TF。 -->
+  <xacro:macro name="ctl_gripper" params="prefix">
+    <joint name="${prefix}gripper">
+      <command_interface name="position">
+        <param name="min">0.0</param>
+        <param name="max">0.1</param>
+      </command_interface>
+      <state_interface name="position"/>
+      <state_interface name="velocity"/>
+      <state_interface name="effort"/>
+    </joint>
+    <joint name="${prefix}gripper_joint1">
+      <state_interface name="position"/>
+      <state_interface name="velocity"/>
+      <state_interface name="effort"/>
+    </joint>
+    <joint name="${prefix}gripper_joint2">
+      <state_interface name="position"/>
+      <state_interface name="velocity"/>
+      <state_interface name="effort"/>
+    </joint>
+  </xacro:macro>
   <ros2_control name="AGRobotSystem" type="system">
     <hardware>
@@ -46,4 +72,6 @@
     <xacro:ctl_arm prefix="arm1_"/>
     <xacro:ctl_arm prefix="arm2_"/>
+    <xacro:ctl_gripper prefix="arm1_"/>
+    <xacro:ctl_gripper prefix="arm2_"/>
   </ros2_control>
   <gazebo>

File: urdf/piper_arm.xacro (robot description, xacro)
@@ -10,5 +10,5 @@
        joint6 速度  5 rad/s      (之前误用 3)
        link2  质量  1.16 kg      (之前 1.17)
-     link6 末端按官方定义挂 flange_link, 再往外是 tool0 安装坐标系(法兰外端面)。
+     link6 末端按官方定义挂 flange_link、tool0 安装坐标系与 PiPER 平行夹爪。
      ===================================================================== -->
 <robot xmlns:xacro="http://www.ros.org/wiki/xacro">
@@ -210,5 +210,5 @@
       <origin xyz="0 0 0" rpy="0 0 0"/>
     </joint>
-    <!-- 末端安装坐标系: 法兰外端面, 以后接夹爪/手爪用这个 frame -->
+    <!-- 末端安装坐标系: 法兰外端面。保留旧 frame 名以兼容现有规划与 TF 用户。 -->
     <link name="${prefix}tool0"/>
     <joint name="${prefix}link6_to_tool0" type="fixed">
@@ -217,4 +217,102 @@
       <origin xyz="0 0 0.0105" rpy="0 0 0"/>
     </joint>
+    <!-- ───────── PiPER 官方平行夹爪 ─────────
+         几何、惯性、安装位姿和限位取自 agx_arm_urdf/piper/
+         urdf/piper_with_gripper_description.xacro。${prefix}gripper 是唯一主动关节，
+         位置值表示两指总开口宽度（0=闭合，0.10 m=全开）；两根指爪通过
+         mimic 分别以 +0.5/-0.5 倍联动。 -->
+    <link name="${prefix}gripper_base">
+      <inertial>
+        <origin xyz="-0.000183807162235591 8.05033155577911E-05 0.0321436689908876" rpy="0 0 0"/>
+        <mass value="0.45"/>
+        <inertia ixx="0.00092934" ixy="0.00000034" ixz="-0.00000738"
+                 iyy="0.00071447" iyz="0.00000005" izz="0.00039442"/>
+      </inertial>
+      <visual>
+        <origin xyz="0 0 0" rpy="0 0 0"/>
+        <geometry><mesh filename="package://ag_robot_description/meshes/piper_gripper_base.dae"/></geometry>
+      </visual>
+      <collision>
+        <origin xyz="0 0 0" rpy="0 0 0"/>
+        <geometry><mesh filename="package://ag_robot_description/meshes/piper_gripper_base.stl"/></geometry>
+      </collision>
+    </link>
+    <joint name="${prefix}gripper_base_joint" type="fixed">
+      <parent link="${prefix}flange_link"/>
+      <child link="${prefix}gripper_base"/>
+      <origin xyz="0 0 0.0045" rpy="0 0 0"/>
+    </joint>
+    <!-- 夹爪驱动器的抽象连杆：无几何，主关节值即总开口宽度。
+         PiPER 官方显示模型把该 link 定义为空 link，但 sdformat 会删除没有
+         inertial 的可动 link，连带删除 gripper 主关节，使后续 mimic 关节
+         找不到驱动源。下面是仅用于保留该仿真自由度的轻量虚拟惯量；
+         官方夹爪实体仍为 0.45 + 0.025 + 0.025 = 0.50 kg。 -->
+    <link name="${prefix}gripper_link">
+      <inertial>
+        <origin xyz="0 0 0" rpy="0 0 0"/>
+        <mass value="0.001"/>
+        <inertia ixx="1.0e-8" ixy="0" ixz="0"
+                 iyy="1.0e-8" iyz="0" izz="1.0e-8"/>
+      </inertial>
+    </link>
+    <joint name="${prefix}gripper" type="prismatic">
+      <parent link="${prefix}gripper_base"/>
+      <child link="${prefix}gripper_link"/>
+      <origin xyz="0 0 0" rpy="0 0 0"/>
+      <axis xyz="0 0 1"/>
+      <limit lower="0" upper="0.1" effort="10" velocity="3"/>
+      <!-- 虚拟驱动关节不加摩擦，实体指爪的阻尼保留在两个 mimic 关节上。 -->
+      <dynamics damping="0" friction="0"/>
+    </joint>
+    <link name="${prefix}gripper_link1">
+      <inertial>
+        <origin xyz="0.00065123185041968 -0.0491929869131989 0.00972258769184025" rpy="0 0 0"/>
+        <mass value="0.025"/>
+        <inertia ixx="0.00007371" ixy="-0.00000113" ixz="0.00000021"
+                 iyy="0.00000781" iyz="-0.00001372" izz="0.0000747"/>
+      </inertial>
+      <visual>
+        <origin xyz="0 0 0" rpy="0 0 0"/>
+        <geometry><mesh filename="package://ag_robot_description/meshes/piper_gripper_link1.dae"/></geometry>
+      </visual>
+      <collision>
+        <origin xyz="0 0 0" rpy="0 0 0"/>
+        <geometry><mesh filename="package://ag_robot_description/meshes/piper_gripper_link1.stl"/></geometry>
+      </collision>
+    </link>
+    <joint name="${prefix}gripper_joint1" type="prismatic">
+      <parent link="${prefix}gripper_base"/>
+      <child link="${prefix}gripper_link1"/>
+      <origin xyz="0 0 0.138" rpy="1.5707963 0 0"/>
+      <axis xyz="0 0 1"/>
+      <limit lower="0" upper="0.05" effort="10" velocity="3"/>
+      <dynamics damping="0.05" friction="0.01"/>
+      <mimic joint="${prefix}gripper" multiplier="0.5" offset="0.0"/>
+    </joint>
+    <link name="${prefix}gripper_link2">
+      <inertial>
+        <origin xyz="0.00065123185041968 -0.0491929869131989 0.00972258769184025" rpy="0 0 0"/>
+        <mass value="0.025"/>
+        <inertia ixx="0.00007371" ixy="-0.00000113" ixz="0.00000021"
+                 iyy="0.00000781" iyz="-0.00001372" izz="0.0000747"/>
+      </inertial>
+      <visual>
+        <origin xyz="0 0 0" rpy="0 0 0"/>
+        <geometry><mesh filename="package://ag_robot_description/meshes/piper_gripper_link2.dae"/></geometry>
+      </visual>
+      <collision>
+        <origin xyz="0 0 0" rpy="0 0 0"/>
+        <geometry><mesh filename="package://ag_robot_description/meshes/piper_gripper_link2.stl"/></geometry>
+      </collision>
+    </link>
+    <joint name="${prefix}gripper_joint2" type="prismatic">
+      <parent link="${prefix}gripper_base"/>
+      <child link="${prefix}gripper_link2"/>
+      <origin xyz="0 0 0.138" rpy="1.5707963 0 -3.1415926"/>
+      <axis xyz="0 0 -1"/>
+      <limit lower="-0.05" upper="0" effort="10" velocity="3"/>
+      <dynamics damping="0.05" friction="0.01"/>
+      <mimic joint="${prefix}gripper" multiplier="-0.5" offset="0.0"/>
+    </joint>
   </xacro:macro>
 </robot>
